File: KiCad_Taffic_Light_Controller/KiCad_Taffic_Light_Controller.kicad_sch (KiCad schematic)
At the start: 50 parts, among them J1 Conn_02x08_Odd_Even, J2 Conn_02x08_Odd_Even, SW1 RST, U1 SM420561N, U2 SM420561N

Commit message: 4/17/26
Parts:
- removed C1, C2: C, symbol Device:C
- removed C3: 0.22u, symbol Device:C
- removed C4: C_Small, symbol Device:C_Small
- added C1: 10u, Capacitor_SMD:CP_Elec_4x5.3, symbol Device:C_Polarized_Small
- added C2, C3: 0.22u, Capacitor_SMD:C_1206_3216Metric_Pad1.33x1.80mm_HandSolder, symbol Device:C_Small
- added C4: 100u, Capacitor_SMD:CP_Elec_6.3x5.8, symbol Device:C_Polarized_Small
- added C5: 0.22U, Capacitor_SMD:C_1206_3216Metric_Pad1.33x1.80mm_HandSolder, symbol Device:C_Small
- added D13: 1N4148W, Diode_SMD:D_SOD-123, symbol Diode:1N4148W
- added H1, H2, H3, H4: MountingHole, MountingHole:MountingHole_2.2mm_M2, symbol Mechanical:MountingHole
- added J3: Control Logic Connector, Connector_PinHeader_2.54mm:PinHeader_2x08_P2.54mm_Vertical, symbol Connector_Generic:Conn_02x05_Odd_Even
- added J4: +5V, my_footprints:Terminal_Block_5mm, symbol Connector:Screw_Terminal_01x02
- added R30, R31, R32: 47K, Resistor_SMD:R_1206_3216Metric_Pad1.30x1.75mm_HandSolder, symbol Device:R
- added SW2: OVR, my_footprints:slide_switch_2.54mm, symbol Switch:SW_SPDT
- added SW3: EN, my_footprints:slide_switch_2.54mm, symbol Switch:SW_SPDT
- added U3: LM1117DT-3.3, Package_TO_SOT_SMD:SOT-223, symbol Regulator_Linear:LM1117DT-3.3
- D1, D10, D2, D3, D4, D5, D6, D7, D8, D9: footprint (none) -> LED_THT:LED_D5.0mm
- J1: value Conn_02x08_Odd_Even -> NS Connector; footprint (none) -> Connector_PinHeader_2.54mm:PinHeader_2x08_P2.54mm_Vertical
- J2: value Conn_02x08_Odd_Even -> EW Connector; footprint (none) -> Connector_PinHeader_2.54mm:PinHeader_2x08_P2.54mm_Vertical
- R1, R10, R11, R12, R13, R14, R15, R16, R17, R18, R19, R2, R20, R21, R22, R23, R24, R25, R26, R27, R28, R29, R3, R4, R5, R6, R7, R8, R9: footprint (none) -> Resistor_SMD:R_1206_3216Metric_Pad1.30x1.75mm_HandSolder
- SW1: footprint (none) -> my_footprints:tact_switch_5mm
Connections:
- net +3.3V: now also C4.1, R30.1, R32.1, U3.2 (VO)
- net GND: now also C1.2, C2.2, C3.2, C4.2, C5.2, J3.10 (Pin_10), J3.2 (Pin_2), J3.4 (Pin_4), J3.6 (Pin_6), J3.8 (Pin_8), J4.2 (Pin_2), SW2.3 (C), SW3.3 (C), U3.1 (GND)
- net RST: now also C3.1, J3.1 (Pin_1)
- net OVR: now reaches D11.1 (K)
- net OVR: now also R28.2, C2.1, J3.5 (Pin_5)
- net at D11.2 (A): now also R28.1, R30.2, SW2.2 (B)
- new net: D13.2 (A), R31.1, R32.2, SW3.2 (B)
- new net +5V: C1.1, J3.7 (Pin_7), J3.9 (Pin_9), J4.1 (Pin_1), U3.3 (VI)
- new net EN: C5.1, D13.1 (K), J3.3 (Pin_3), R31.2
Other:
- note added: "+3.3V VOLTAGE REGULATOR"
- note added: "CONTROL LOGIC"
- note added: "EMERGENCY OVERRIDE"
- note added: "ENABLE"
- note added: "MOUNTING HOLES"
- moved on the sheet: D11, R28

Commit message: 4/19(1pm)
Parts:
- J3: footprint Connector_PinHeader_2.54mm:PinHeader_2x08_P2.54mm_Vertical -> Connector_PinHeader_2.54mm:PinHeader_2x05_P2.54mm_Vertical
Connections:
- net +5V: no longer C1.1, U3.3 (VI)
- net x: now reaches SW3.1 (A)
- net x: now also SW2.1 (A)
- new net: C1.1, U3.3 (VI)

Commit message: 5:23PM
Parts:
- D10, D8: value NSC_YLW -> NSC_RED
Connections:
- net +5V: now also C1.1, U3.3 (VI)
Changed lines of the file:
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@@
 	)
 	(junction
+		(at 208.28 119.38)
+		(diameter 0)
+		(color 0 0 0 0)
+	)
+	(junction
 		(at 73.66 44.45)
 		(diameter 0)
@@
 	)
 	(junction
-		(at 208.28 119.38)
-		(diameter 0)
-		(color 0 0 0 0)
-	)
-	(junction
 		(at 266.7 88.9)
 		(diameter 0)
@@
 	(wire
 		(pts
-			(xy 205.74 119.38) (xy 208.28 119.38)
-		)
-		(stroke
-			(width 0)
-			(type default)
-		)
-	)
-	(wire
-		(pts
 			(xy 259.08 39.37) (xy 261.62 39.37)
 		)
@@
 	(wire
 		(pts
-			(xy 210.82 119.38) (xy 208.28 119.38)
-		)
-		(stroke
-			(width 0)
-			(type default)
-		)
-	)
-	(wire
-		(pts
 			(xy 29.21 105.41) (xy 34.29 105.41)
 		)
@@
 	(wire
 		(pts
+			(xy 208.28 119.38) (xy 210.82 119.38)
+		)
+		(stroke
+			(width 0)
+			(type default)
+		)
+	)
+	(wire
+		(pts
 			(xy 276.86 41.91) (xy 276.86 53.34)
 		)
@@
 	(wire
 		(pts
+			(xy 208.28 119.38) (xy 208.28 121.92)
+		)
+		(stroke
+			(width 0)
+			(type default)
+		)
+	)
+	(wire
+		(pts
 			(xy 83.82 88.9) (xy 88.9 88.9)
 		)
@@
 	(wire
 		(pts
-			(xy 208.28 119.38) (xy 208.28 121.92)
+			(xy 262.89 91.44) (xy 266.7 91.44)
 		)
 		(stroke
@@
 	(wire
 		(pts
-			(xy 262.89 91.44) (xy 266.7 91.44)
+			(xy 226.06 119.38) (xy 228.6 119.38)
 		)
 		(stroke
@@
 	(wire
 		(pts
-			(xy 226.06 119.38) (xy 228.6 119.38)
+			(xy 41.91 55.88) (xy 45.72 55.88)
 		)
 		(stroke
@@
 	(wire
 		(pts
-			(xy 41.91 55.88) (xy 45.72 55.88)
+			(xy 266.7 88.9) (xy 266.7 91.44)
 		)
 		(stroke
@@
 	(wire
 		(pts
-			(xy 266.7 88.9) (xy 266.7 91.44)
+			(xy 76.2 34.29) (xy 73.66 34.29)
 		)
 		(stroke
@@
 	(wire
 		(pts
-			(xy 76.2 34.29) (xy 73.66 34.29)
+			(xy 205.74 119.38) (xy 208.28 119.38)
 		)
 		(stroke
@@
 		)
 	)
+	(label "+5V"
+		(at 205.74 119.38 180)
+		(effects
+			(font
+				(size 1.27 1.27)
+			)
+			(justify right bottom)
+		)
+	)
 	(label "NS_HEX_C"
 		(at 29.21 97.79 180)
@@
 	)
 	(symbol
+		(lib_id "power:PWR_FLAG")
+		(at 205.74 119.38 90)
+		(unit 1)
+		(exclude_from_sim no)
+		(in_bom yes)
+		(on_board yes)
+		(dnp no)
+		(fields_autoplaced yes)
+		(property "Reference" "#FLG01"
+			(at 203.835 119.38 0)
+			(effects
+				(font
+					(size 1.27 1.27)
+				)
+				(hide yes)
+			)
+		)
+		(property "Value" "PWR_FLAG"
+			(at 200.66 119.38 0)
+			(effects
+				(font
+					(size 1.27 1.27)
+				)
+				(hide yes)
+			)
+		)
+		(property "Footprint" ""
+			(at 205.74 119.38 0)
+			(effects
+				(font
+					(size 1.27 1.27)
+				)
+				(hide yes)
+			)
+		)
+		(property "Datasheet" "~"
+			(at 205.74 119.38 0)
+			(effects
+				(font
+					(size 1.27 1.27)
+				)
+				(hide yes)
+			)
+		)
+		(property "Description" "Special symbol for telling ERC where power comes from"
+			(at 205.74 119.38 0)
+			(effects
+				(font
+					(size 1.27 1.27)
+				)
+				(hide yes)
+			)
+		)
+		(pin "1"
+		)
+		(instances
+			(project ""
+				(path "/be8e9ab3-66fc-4eb3-b7df-696c5fd901b8"
+					(reference "#FLG01")
+					(unit 1)
+				)
+			)
+		)
+	)
+	(symbol
 		(lib_id "Device:R")
 		(at 123.19 44.45 270)
@@
 			)
 		)
-		(property "Value" "NSC_YLW"
+		(property "Value" "NSC_RED"
 			(at 134.62 96.52 0)
 			(effects
@@
 	)
 	(symbol
-		(lib_id "power:PWR_FLAG")
-		(at 205.74 119.38 0)
-		(unit 1)
-		(exclude_from_sim no)
-		(in_bom yes)
-		(on_board yes)
-		(dnp no)
-		(property "Reference" "#FLG01"
-			(at 205.74 117.475 0)
-			(effects
-				(font
-					(size 1.27 1.27)
-				)
-				(hide yes)
-			)
-		)
-		(property "Value" "+5V"
-			(at 202.692 119.38 0)
-			(effects
-				(font
-					(size 1.27 1.27)
-				)
-			)
-		)
-		(property "Footprint" ""
-			(at 205.74 119.38 0)
-			(effects
-				(font
-					(size 1.27 1.27)
-				)
-				(hide yes)
-			)
-		)
-		(property "Datasheet" "~"
-			(at 205.74 119.38 0)
-			(effects
-				(font
-					(size 1.27 1.27)
-				)
-				(hide yes)
-			)
-		)
-		(property "Description" "Special symbol for telling ERC where power comes from"
-			(at 205.74 119.38 0)
-			(effects
-				(font
-					(size 1.27 1.27)
-				)
-				(hide yes)
-			)
-		)
-		(pin "1"
-		)
-		(instances
-			(project ""
-				(path "/be8e9ab3-66fc-4eb3-b7df-696c5fd901b8"
-					(reference "#FLG01")
-					(unit 1)
-				)
-			)
-		)
-	)
-	(symbol
 		(lib_id "Diode:1N4148W")
 		(at 223.52 40.64 180)
@@
 			)
 		)
-		(property "Value" "NSC_YLW"
+		(property "Value" "NSC_RED"
 			(at 134.62 41.656 0)
 			(effects
