File: KiCad_Taffic_Light_Controller/KiCad_Taffic_Light_Controller.kicad_pcb (KiCad board)
At the start: 2 copper layers, 64 parts, among them J1 NS Connector, J2 EW Connector, J3 Control Logic Connector, J4 +5V, SW1 RST, SW2 OVR, SW3 EN, U1 SM420561N, U2 SM420561N, U3 LM1117DT-3.3

Commit message: 5:23PM
Parts:
- D10, D8: value NSC_YLW -> NSC_RED
- moved H1 137.3 mm to (20.5, 167.7)
- moved H3 137.3 mm to (20.5, 179.6)
- moved H2 137.3 mm to (20.5, 173.6)
- moved H4 137.3 mm to (20.5, 185.5)
- moved R7 118.1 mm to (167.1, 53.1), turned to 90 degrees
- moved R6 116.4 mm to (171.1, 53.1), turned to 90 degrees
- moved R17 115.1 mm to (148.6, 54.1)
- moved R23 112.3 mm to (199.1, 62.1)
- moved R2 107.5 mm to (179.1, 53.1), turned to 90 degrees
- moved R18 107.4 mm to (148.6, 65.1)
- moved R24 106.2 mm to (199.1, 72.6)
- moved R1 102.8 mm to (175.1, 53.1), turned to 90 degrees
- moved R8 99.5 mm to (179.1, 82.1), turned to -90 degrees
- moved J3 94.7 mm to (123.8, 54.5), turned to 90 degrees
- moved R27 89.4 mm to (192.0, 98.0)
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Connections:
- C1 pad 1: Net-(U3-VI) -> /+5V
- U3 pad 3: Net-(U3-VI) -> /+5V
Other:
- board text added: "+3.3V"
- board text added: "A"
- board text added: "B"
- board text added: "C"
- board text added: "CAR"
- board text added: "D"
- board text added: "DP"
- board text added: "E"
- board text added: "EN"
- board text added: "F"
- board text added: "G"
- board text added: "GND"
- board text added: "OVR"
- board text added: "PED"
- board text added: "R"
- board text added: "RST"
- board text added: "Y"

Commit message: hala
Parts:
- moved C1 1.92 mm to (103.0, 75.6)
- moved C4 1.92 mm to (104.0, 66.6)
- turned C2 to 180 degrees
- turned C3 to 180 degrees
- turned C5 to 180 degrees
- turned D11 to 180 degrees
- turned D12 to 180 degrees
- turned D13 to 180 degrees
- turned R17 to 180 degrees
- turned R18 to 180 degrees
- turned R19 to 180 degrees
- turned R27 to 180 degrees
- turned R29 to 180 degrees
- turned R30 to 180 degrees
- turned R32 to 180 degrees
Connections:
- J4 pad 1: /+5V -> GND
- J4 pad 2: GND -> /+5V
Routing:
- net GND: track 0.00 -> 244.3 mm
- net /+3.3V: track 0.00 -> 100.4 mm, vias 0 -> 1
- net /NS_HEX_F: track 0.00 -> 96.7 mm
- net /NS_HEX_G: track 0.00 -> 93.6 mm
- net /NS_HEX_D: track 0.00 -> 92.6 mm
- net /+5V: track 0.00 -> 89.8 mm
- net /NS_HEX_C: track 0.00 -> 86.1 mm
- net /NS_HEX_E: track 0.00 -> 81.3 mm, vias 0 -> 1
- net /NS_HEX_DP: track 0.00 -> 76.6 mm, vias 0 -> 1
- net /NSP_RED: track 0.00 -> 71.1 mm
- net /NSP_GRN: track 0.00 -> 51.5 mm
- net /NS_HEX_A: track 0.00 -> 23.2 mm
- net /NS_HEX_B: track 0.00 -> 22.6 mm
- net Net-(D13-A): track 0.00 -> 14.2 mm
- net Net-(D12-A): track 0.00 -> 12.1 mm
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